Commit message: better forces

File: resources/urdf/franka_panda/panda_robotiq_noinertia.urdf (robot description, URDF)
Before this commit: robot panda, 21 links, 20 joints
Links:
- link panda_link1: mass 2.7 -> None
- link panda_link2: mass 2.73 -> None
- link panda_link3: mass 2.04 -> None
- link panda_link4: mass 2.08 -> None
- link panda_link5: mass 3 -> None
- link panda_link6: mass 1.3 -> None
- link panda_link7: mass .2 -> None
- link panda_link8: mass 0.0 -> None
- link robotiq_2f_85_left_inner_finger_pad: mass 0.0 -> None
- link robotiq_2f_85_right_inner_finger_pad: mass 0.0 -> None
- link robotiq_85_base_link: mass 0.0 -> 0.22652
- link robotiq_85_coupling_link: mass 0.0 -> None
- link robotiq_85_left_finger_link: mass 0.027309 -> None
- link robotiq_85_left_finger_tip_link: mass 0.019555 -> None
- link robotiq_85_left_inner_knuckle_link: mass 0.029951 -> None
- link robotiq_85_left_knuckle_link: mass 0.018491 -> None
- link robotiq_85_right_finger_link: mass 0.027309 -> None
- link robotiq_85_right_finger_tip_link: mass 0.019555 -> None
- link robotiq_85_right_inner_knuckle_link: mass 0.029951 -> None
- link robotiq_85_right_knuckle_link: mass 0.018491 -> None
